File: motor_controllers.kicad_sch (KiCad schematic)
At the start: 31 parts, among them IC3 L6470H, IC4 L6470H, IC5 74AUP2G00DC,125

Commit message: Updated ADCs resistor value
Parts:
- R19, R21: value 27k -> 150k
