File: rpiboard_minirys.kicad_pcb (KiCad board)
At the start: 4 copper layers, 65 x 56 mm, 132 parts, among them IC1 LM51231QRGRRQ1, IC2 TPS564242DRLR, IC3 L6470H, IC4 L6470H, IC5 74AUP2G00DC,125, IC6 MAX11613EUA+T, J1 RPi_GPIO, J10 ToF1_Sensor, J11 ToF2_Sensor, J12 ToF3_Sensor, J13 ToF4_Sensor, J14 ToF5_Sensor, J15 ToF6_Sensor, J16 SPI_Connector, J17 UART_Connector, J18 Fan_Connector, J2 Motor_L, J3 Motor_R, J4 B_Cell_3, J5 B_Cell_2, J6 B_Cell_1, J7 SW, J8 Temp_Sensor, J9 IMU_Sensor, Q1 DMG1012T-7, Q2 ISZ065N03L5S, Q3 ISZ065N03L5S, Q4 DMG1012T-7, Q5 DMG1012T-7, Q6 DMG1012T-7

Commit message: Updated ADCs resistor value
Parts:
- R19, R21: value 27k -> 150k
Changed lines of the file:
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@@
         (effects (font (size 1 1) (thickness 0.2) bold))
     )
-    (fp_text value "27k" (at 0 1.43 90) (layer "F.Fab")
+    (fp_text value "150k" (at 0 1.43 90) (layer "F.Fab")
         (effects (font (size 1 1) (thickness 0.15)))
     )
@@
         (effects (font (size 1 1) (thickness 0.2)))
     )
-    (fp_text value "27k" (at 0 1.43 90) (layer "F.Fab")
-        (effects (font (size 1 1) (thickness 0.15)))
-    )
+    (fp_text value "150k" (at 0 1.43 90) (layer "F.Fab")
+        (effects (font (size 1 1) (thickness 0.15)))
+    )
